File: esquema_mux_comedero/esquema_mux_comedero.kicad_sch (KiCad schematic)
At the start: 3 parts

Commit message: 2 sense
Parts:
- added U2: ~, symbol Mensoft_Carmen:SN74HC4851N
- renumbered U6 to U1
Connections:
- net +3.3V: now also U2.16 (Vcc)
- net GNDREF: now also U2.8 (GND)
- net Pin 13: now also U2.3 (COM); no longer U1.2 (RX), U2.2 (RX)
- net Pin 18: now also U2.11 (A)
- net Pin 22: now also U2.9 (C)
- net Pin 23: now also U2.6 (INH)
- net Pin 5: now also U2.10 (B)
- new net: U1.2 (RX), U2.13 (Y0)
- new net: U2.14 (Y1), U2.2 (RX)
- no-connect marks 3 -> 6
Other:
- moved on the sheet: U1, U2

Commit message: 1mux
Parts:
- removed U2: ~, symbol Mensoft_Carmen:SN74HC4851N
- renumbered U1 to U3
Connections:
- net Pin 13: now also U1.2 (RX), U2.2 (RX)
- no-connect marks 6 -> 7
Other:
- moved on the sheet: U1, U2

Commit message: pin18
Connections:
- net Pin 13 is gone; now on net Pin 19: U1.2 (RX), U2.2 (RX)
- net Pin 18: now also U3.3 (COM)
- net Pin 19: no longer U3.3 (COM)
Other:
- note added: "Pin 19: MISO Pin 5: SD_CS Pin 18: CLK Pin 22: SCL Pin 23: MOSI"
- note removed: "Pin 13: SENSE1 Pin 19: MISO Pin 5: SD_CS Pin 18: CLK Pin 22: SCL Pin 23: MOSI"
Changed lines of the file:
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@@
 	(bus
 		(pts
-			(xy 140.97 60.96) (xy 158.75 60.96)
+			(xy 138.43 64.77) (xy 156.21 64.77)
 		)
 		(stroke
@@
 	(bus
 		(pts
-			(xy 140.97 77.47) (xy 158.75 77.47)
+			(xy 138.43 81.28) (xy 156.21 81.28)
 		)
 		(stroke
@@
 	(bus
 		(pts
-			(xy 140.97 60.96) (xy 140.97 77.47)
+			(xy 138.43 64.77) (xy 138.43 81.28)
 		)
 		(stroke
@@
 	(bus
 		(pts
-			(xy 158.75 77.47) (xy 158.75 60.96)
+			(xy 156.21 81.28) (xy 156.21 64.77)
 		)
 		(stroke
@@
 		)
 	)
-	(text "Pin 13: SENSE1\nPin 19: MISO\n\nPin 5: SD_CS\nPin 18: CLK\nPin 22: SCL\nPin 23: MOSI\n"
+	(text "Pin 19: MISO\n\nPin 5: SD_CS\nPin 18: CLK\nPin 22: SCL\nPin 23: MOSI\n"
 		(exclude_from_sim no)
-		(at 150.368 69.088 0)
+		(at 147.828 72.898 0)
 		(effects
 			(font
@@
 		)
 	)
-	(global_label "Pin 13"
+	(global_label "Pin 19"
 		(shape input)
 		(at 101.6 99.06 270)
@@
 		)
 	)
+	(global_label "Pin 18"
+		(shape input)
+		(at 96.52 151.13 270)
+		(fields_autoplaced yes)
+		(effects
+			(font
+				(size 1.27 1.27)
+				(thickness 0.254)
+				(bold yes)
+				(color 0 0 72 1)
+			)
+			(justify right)
+		)
+		(property "Intersheetrefs" "${INTERSHEET_REFS}"
+			(at 96.52 161.0016 90)
+			(effects
+				(font
+					(size 1.27 1.27)
+				)
+				(justify right)
+				(hide yes)
+			)
+		)
+	)
+	(global_label "Pin 18"
+		(shape input)
+		(at 111.76 124.46 90)
+		(fields_autoplaced yes)
+		(effects
+			(font
+				(size 1.27 1.27)
+				(thickness 0.254)
+				(bold yes)
+				(color 0 0 72 1)
+			)
+			(justify left)
+		)
+		(property "Intersheetrefs" "${INTERSHEET_REFS}"
+			(at 111.76 114.5884 90)
+			(effects
+				(font
+					(size 1.27 1.27)
+				)
+				(justify left)
+				(hide yes)
+			)
+		)
+	)
+	(global_label "Pin 22"
+		(shape input)
+		(at 121.92 124.46 90)
+		(fields_autoplaced yes)
+		(effects
+			(font
+				(size 1.27 1.27)
+				(thickness 0.254)
+				(bold yes)
+				(color 194 0 194 1)
+			)
+			(justify left)
+		)
+		(property "Intersheetrefs" "${INTERSHEET_REFS}"
+			(at 121.92 114.5884 90)
+			(effects
+				(font
+					(size 1.27 1.27)
+				)
+				(justify left)
+				(hide yes)
+			)
+		)
+	)
 	(global_label "Pin 19"
 		(shape input)
-		(at 96.52 151.13 270)
-		(fields_autoplaced yes)
-		(effects
-			(font
-				(size 1.27 1.27)
-				(thickness 0.254)
-				(bold yes)
-				(color 0 0 72 1)
-			)
-			(justify right)
-		)
-		(property "Intersheetrefs" "${INTERSHEET_REFS}"
-			(at 96.52 161.0016 90)
-			(effects
-				(font
-					(size 1.27 1.27)
-				)
-				(justify right)
-				(hide yes)
-			)
-		)
-	)
-	(global_label "Pin 18"
-		(shape input)
-		(at 111.76 124.46 90)
-		(fields_autoplaced yes)
-		(effects
-			(font
-				(size 1.27 1.27)
-				(thickness 0.254)
-				(bold yes)
-				(color 0 0 72 1)
-			)
-			(justify left)
-		)
-		(property "Intersheetrefs" "${INTERSHEET_REFS}"
-			(at 111.76 114.5884 90)
-			(effects
-				(font
-					(size 1.27 1.27)
-				)
-				(justify left)
-				(hide yes)
-			)
-		)
-	)
-	(global_label "Pin 22"
-		(shape input)
-		(at 121.92 124.46 90)
-		(fields_autoplaced yes)
-		(effects
-			(font
-				(size 1.27 1.27)
-				(thickness 0.254)
-				(bold yes)
-				(color 194 0 194 1)
-			)
-			(justify left)
-		)
-		(property "Intersheetrefs" "${INTERSHEET_REFS}"
-			(at 121.92 114.5884 90)
-			(effects
-				(font
-					(size 1.27 1.27)
-				)
-				(justify left)
-				(hide yes)
-			)
-		)
-	)
-	(global_label "Pin 13"
-		(shape input)
 		(at 147.32 110.49 270)
