File: esquema_mux_comedero/esquema_mux_comedero.kicad_sch (KiCad schematic)
At the start: 7 parts

Commit message: sket
Connections:
- net GNDREF: now also U1.3 (GND), U2.3 (GND), U3.3 (GND), U4.3 (GND), U5.3 (GND); no longer U6.6 (INH), U7.6 (INH)
- net Pin 23: now also U6.6 (INH), U7.6 (INH); no longer U1.3 (GND), U2.3 (GND), U3.3 (GND), U4.3 (GND), U5.3 (GND)

Commit message: nc
Connections:
- net GNDREF: now also U7.7 (NC)
Changed lines of the file:
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@@
 	(generator_version "8.0")
 	(paper "A4")
+	(junction
+		(at 220.98 119.38)
+		(diameter 0)
+		(color 0 0 0 0)
+	)
 	(no_connect
 		(at 78.74 119.38)
@@
 	(wire
 		(pts
+			(xy 220.98 119.38) (xy 220.98 120.65)
+		)
+		(stroke
+			(width 0)
+			(type default)
+		)
+	)
+	(wire
+		(pts
 			(xy 63.5 119.38) (xy 63.5 116.84)
 		)
@@
 	(wire
 		(pts
-			(xy 220.98 116.84) (xy 220.98 120.65)
+			(xy 220.98 116.84) (xy 220.98 119.38)
 		)
 		(stroke
@@
 	(wire
 		(pts
+			(xy 215.9 116.84) (xy 215.9 119.38)
+		)
+		(stroke
+			(width 0)
+			(type default)
+		)
+	)
+	(wire
+		(pts
 			(xy 215.9 93.98) (xy 215.9 96.52)
 		)
@@
 		)
 		(stroke
+			(width 0)
+			(type default)
+		)
+	)
+	(wire
+		(pts
+			(xy 215.9 119.38) (xy 220.98 119.38)
+		)
+		(stroke

Commit message: opt
Parts:
- removed U7: ~, symbol Mensoft_Carmen:SN74HC4851N
Connections:
- net GNDREF: now also U6.7 (NC)
- net Pin 18: now also U6.3 (COM)
- net Pin 19: now also U1.2 (RX), U2.2 (RX), U3.2 (RX), U4.2 (RX), U5.2 (RX); no longer U6.3 (COM)
- no-connect marks 6 -> 3
Other:
- moved on the sheet: U1, U2, U3, U4, U5, U6

Commit message: opt final
Connections:
- net Pin 13 is gone; now on net Pin 18: U6.11 (A)
- net GNDREF: now also U1.2 (RX), U2.2 (RX), U3.2 (RX), U4.2 (RX), U5.2 (RX)
- net Pin 18: no longer U6.3 (COM)
- net Pin 19: now also U6.3 (COM); no longer U1.2 (RX), U2.2 (RX), U3.2 (RX), U4.2 (RX), U5.2 (RX)
- net Pin 14 renamed Pin 22
- net Pin 15 renamed Pin 5
Other:
- note added: "Pin 19: MISO Pin 23: MOSI Pin 5: SD_CS Pin 18: CLK Pin 22: SCL"
- note removed: "Pin 13: SENSE1 Pin 14: SENSE3 Pin 15: SENSE2 Pin 18: CLK Pin 19: MISO Pin 23: MOSI"
